File: Chord Board Controller.kicad_sch (KiCad schematic)
At the start: 62 parts, among them J4 HRO_TYPE-C-31-M-14, J6 TC2030_SWD, J8 Battery, Q13 2N7002, SW6 SW_SPST, SW7 RST, SW8 SW_SPDT, U5 SRV05-4, U6 XC6206PxxxMR, U7 nRF52840_holyiot_18010, U8 BQ24075RGT

Commit message: cc Text
Other:
- note added: "CHord controller"
Changed lines of the file:
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@@
+		)
+	)
+	(text "CHord controller"
+		(exclude_from_sim no)
+		(at 318.008 208.788 0)
+		(effects
+			(font
+				(size 2.54 2.54)
+			)
 		)
 	)
